Commit message: Add joint_trans and robot_chassis_controller.

File: catkin_ws/src/learn_description/urdf/robot.xacro (robot description, xacro)
@@ -1,3 +1,3 @@
-<robot name="robot">
+<robot name="robot" xmlns:xacro="http://wiki.ros.org/xacro">
     <link name="base_footprint">
         <visual>
@@ -17,5 +17,5 @@
             <origin xyz="0 0 0"/>
             <mass value="6" />
-            <inertia ixx="1" ixy="0" ixz="0" iyy="1" iyz="0" izz="1" />
+            <inertia ixx="0.185" ixy="0" ixz="0" iyy="0.2" iyz="0" izz="0.025" />
         </inertial>
         <collision>
@@ -56,5 +56,5 @@
             <origin xyz="0 0 0"/>
             <mass value="2" />
-            <inertia ixx="1" ixy="0" ixz="0" iyy="1" iyz="0" izz="1" />
+            <inertia ixx="3.8e-3" ixy="0" ixz="0" iyy="3.8e-3" iyz="0" izz="6.4e-3" />
         </inertial>
         <collision>
@@ -81,5 +81,5 @@
             <origin xyz="0 0 0"/>
             <mass value="2" />
-            <inertia ixx="1" ixy="0" ixz="0" iyy="1" iyz="0" izz="1" />
+            <inertia ixx="3.8e-3" ixy="0" ixz="0" iyy="3.8e-3" iyz="0" izz="6.4e-3" />
         </inertial>
         <collision>
@@ -106,5 +106,5 @@
             <origin xyz="0 0 0"/>
             <mass value="2" />
-            <inertia ixx="1" ixy="0" ixz="0" iyy="1" iyz="0" izz="1" />
+            <inertia ixx="3.8e-3" ixy="0" ixz="0" iyy="3.8e-3" iyz="0" izz="6.4e-3" />
         </inertial>
         <collision>
@@ -131,5 +131,5 @@
             <origin xyz="0 0 0"/>
             <mass value="2" />
-            <inertia ixx="1" ixy="0" ixz="0" iyy="1" iyz="0" izz="1" />
+            <inertia ixx="3.8e-3" ixy="0" ixz="0" iyy="3.8e-3" iyz="0" izz="6.4e-3" />
         </inertial>
         <collision>
@@ -146,3 +146,25 @@
         <axis xyz="0 1 0" />
     </joint>
+    <xacro:macro name="joint_trans" params="joint_name">
+        <!-- Transmission is important to link the joints and the controller -->
+        <transmission name="${joint_name}_trans">
+            <type>transmission_interface/SimpleTransmission</type>
+            <joint name="${joint_name}_joint">
+                <hardwareInterface>hardware_interface/VelocityJointInterface</hardwareInterface>
+            </joint>
+            <actuator name="${joint_name}_motor">
+                <hardwareInterface>hardware_interface/VelocityJointInterface</hardwareInterface>
+                <mechanicalReduction>1</mechanicalReduction>
+            </actuator>
+        </transmission>
+    </xacro:macro>
+    <xacro:joint_trans joint_name="left_front_wheel" />
+    <xacro:joint_trans joint_name="left_back_wheel" />
+    <xacro:joint_trans joint_name="right_front_wheel" />
+    <xacro:joint_trans joint_name="right_back_wheel" />
+    <gazebo>
+        <plugin name="ros_control" filename="libgazebo_ros_control.so">
+            <robotNamespace>/</robotNamespace>
+        </plugin>
+    </gazebo>
 </robot>

Commit message: Update rosbot_description.

File: catkin_ws/src/learn_description/urdf/robot.xacro (robot description, xacro)
@@ -1,10 +1,7 @@
 <robot name="robot" xmlns:xacro="http://wiki.ros.org/xacro">
-    <link name="base_footprint">
-        <visual>
-            <geometry>
-                <sphere radius="0.001" />
-            </geometry>
-        </visual>
-    </link>
+    <xacro:property name="wheel_radius" value="0.08" />
+    <xacro:property name="chassis_length" value="0.6" />
+    <xacro:property name="chassis_width" value="0.2" />
+    <xacro:property name="chassis_height" value="0.1" />
     <link name="base_link">
         <visual>
@@ -41,9 +38,4 @@
         <material>Gazebo/Black</material>
     </gazebo>
-    <joint name="base_link2base_footprint" type="fixed">
-        <parent link="base_footprint" />
-        <child link="base_link"/>
-        <origin xyz="0 0 0.2" />
-    </joint>
     <link name="left_front_wheel">
         <visual>
