Commit message: Finish urdf_learn.md and improve the code.

File: my_robot/urdf/robot.urdf.xacro (robot description, xacro)
@@ -25,5 +25,5 @@
         </collision>
         <inertial>
-            <mass value="1.0"/>
+            <mass value="10.0"/>
             <inertia ixx="1.042" ixy="0.0" ixz="0.0" iyy="3.542" iyz="0.0" izz="4.167"/>
         </inertial>
